File: Rocky Switch Shield.brd (EAGLE design)
At the start: 68.4 x 47 mm, 14 parts

Commit message: Update new shield for rocky switch
Parts:
- removed CAP_BTN1, CAP_BTN2, CAP_BTN3: (no value), adafruit:1X03
- removed JP2: (no value), adafruit:2X04
- added B5, B6, B7, B8: (no value), PatternAgents-TouchWidgets:BUTTON_PASSIVE_12MM
- added C1, C3, C5, C7: 30pF, rcl:C0805K
- added C2, C4, C6, C8: 0.1uF, rcl:C0805K
- added JP1: (no value), pinhead:2X05
- added LED4: (no value), adafruit:LED3MM
- added R4: 1K, rcl:R0805
- added SJ1, SJ2, SJ3, SJ4, SJ5, SJ6, SJ7, SJ8: JUMPER-PAD-2-NOYES_SILK, SparkFun-Passives:PAD-JUMPER-2-NO_YES_SILK
- added U$1, U$2, U$3, U$4: TTP223B, My Eagle Lib:SOT23-6
- moved LED2 45.8 mm to (18.4, 36.2), turned to 180 degrees
- moved R3 44.4 mm to (50.8, 8.89)
- moved LED3 44.1 mm to (50.8, 14.0), turned to 180 degrees
- moved R1 43.5 mm to (18.4, 8.89)
- moved LED1 42.8 mm to (18.4, 14.0), turned to 180 degrees
- moved R2 41.5 mm to (18.4, 30.5), turned to 180 degrees
- moved U$6 40.2 mm to (4.19, 2.92)
- moved U$9 37.6 mm to (4.19, 47.1)
- moved U$7 34.6 mm to (77.9, 2.92)
- moved U$8 31.6 mm to (77.9, 47.1)
Connections:
- removed net 3V3: CAP_BTN1.3, CAP_BTN2.3, CAP_BTN3.3, JP2.1
- new net D3: JP1.6, LED3.K
- new net D4: JP1.8, LED4.K
- new net I1: B5.BUTTON, C1.1, U$1.3
- new net I2: B6.BUTTON, C3.1, U$2.3
- new net I3: B7.BUTTON, C5.1, U$3.3
- new net I4: B8.BUTTON, C7.1, U$4.3
- new net N$1: SJ1.1, U$1.4
- new net N$11: SJ5.1, U$3.4
- new net N$12: SJ6.1, U$3.6
- new net N$15: SJ7.1, U$4.4
- new net N$16: SJ8.1, U$4.6
- new net N$5: SJ2.1, U$1.6
- new net N$7: SJ3.1, U$2.4
- new net N$8: SJ4.1, U$2.6
- new net N$9: LED4.A, R4.2
- new net VDD: C2.1, C4.1, C6.1, C8.1, JP1.10, R1.1, R2.1, R3.1, R4.1, SJ1.2, SJ2.2, SJ3.2, SJ4.2, SJ5.2, SJ6.2, SJ7.2, SJ8.2, U$1.5, U$2.5, U$3.5, U$4.5
- net D0: now also JP1.7, U$1.1; no longer CAP_BTN1.2, JP2.4
- net D1: now also JP1.2, LED1.K; no longer CAP_BTN2.2, JP2.6
- net D2: now also JP1.4, LED2.K; no longer CAP_BTN3.2, JP2.8
- net D5: now also JP1.5, U$2.1; no longer JP2.7, R3.1
- net D6: now also JP1.3, U$3.1; no longer JP2.5, R2.1
- net D7: now also JP1.1, U$4.1; no longer JP2.3, R1.1
- net GND: now also C1.2, C2.2, C3.2, C4.2, C5.2, C6.2, C7.2, C8.2, JP1.9, U$1.2, U$2.2, U$3.2, U$4.2; no longer CAP_BTN1.1, CAP_BTN2.1, CAP_BTN3.1, JP2.2, LED1.K, LED2.K, LED3.K
Routing:
- net VDD: track 0.00 -> 150.5 mm
- net 3V3: track 54.4 -> 0.00 mm
- net D3: track 0.00 -> 53.9 mm
- net D4: track 0.00 -> 52.9 mm
- net GND: track 72.9 -> 125.8 mm, vias 0 -> 1
- net D7: track 22.9 -> 64.0 mm, vias 0 -> 1
- net D2: track 52.5 -> 20.1 mm
- net D5: track 57.3 -> 31.8 mm
- net D1: track 35.5 -> 18.3 mm
- net D0: track 16.2 -> 31.2 mm, vias 0 -> 1
- net I3: track 0.00 -> 13.2 mm
- net I1: track 0.00 -> 13.0 mm
- net I2: track 0.00 -> 13.0 mm
- net I4: track 0.00 -> 13.0 mm
- net N$9: track 0.00 -> 5.85 mm
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Other:
- board size 68.4 x 47 mm -> 81.1 x 50.2 mm
- board text added: "5V"
- board text added: "D3"
- board text added: "D4"
- board text removed: "3V3"
- board text removed: "Touch"

Commit message: Update board design to version 0.2
Parts:
- LED1, LED2, LED3, LED4: device adafruit:LED3MM -> adafruit:CHIP-LED0805
- SJ1, SJ3, SJ5, SJ7: value JUMPER-PAD-2-NOYES_SILK -> AHLB
- SJ2, SJ4, SJ6, SJ8: value JUMPER-PAD-2-NOYES_SILK -> TOG
- moved U$7 9.15 mm to (69.6, 6.86)
- moved U$8 8.53 mm to (69.6, 49.3)
- moved JP1 7.24 mm to (6.99, 38.1)
- moved B7 5.68 mm to (57.1, 16.5)
- moved R4 5.68 mm to (45.7, 33.0)
- moved SJ5 5.68 mm to (42.5, 23.5)
- moved B8 5.68 mm to (57.1, 38.7)
- moved C5 5.68 mm to (47.0, 20.3)
- moved C6 5.68 mm to (42.5, 20.3)
- moved C7 5.68 mm to (47.0, 43.2)
- moved C8 5.68 mm to (42.5, 43.2)
- moved R3 5.68 mm to (45.7, 11.4)
- moved SJ6 5.68 mm to (42.5, 26.0)
- moved SJ7 5.68 mm to (42.5, 45.7)
- moved SJ8 5.68 mm to (42.5, 48.3)
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Connections:
- net D1: now also LED1.C; no longer LED1.K
- net D2: now also LED2.C; no longer LED2.K
- net D3: now also LED3.C; no longer LED3.K
- net D4: now also LED4.C; no longer LED4.K
Routing:
- net D3: track 53.9 -> 68.7 mm
- net D5: track 31.8 -> 23.2 mm, vias 0 -> 1
- net VDD: track 150.5 -> 142.5 mm, vias 0 -> 2
- net D0: track 31.2 -> 25.1 mm, vias 1 -> 0
- net D2: track 20.1 -> 25.6 mm, vias 0 -> 1
- net D4: track 52.9 -> 57.4 mm
- net D6: track 49.3 -> 45.4 mm
- net D1: track 18.3 -> 21.8 mm
- net D7: track 64.0 -> 61.4 mm
- net N$9: track 5.85 -> 5.33 mm, vias 0 -> 1
- net N$6: track 5.21 -> 4.69 mm, vias 0 -> 1
- net N$3: track 5.21 -> 4.69 mm, vias 0 -> 1
- net I3: track 13.2 -> 12.7 mm
- net N$4: track 5.85 -> 5.68 mm, vias 0 -> 1
Other:
- board size 81.1 x 50.2 mm -> 69.6 x 47.6 mm
- board text added: "Rocky Switch Shield v0.2"
- board text removed: "Rocky Switch Shield"

Commit message: Update design to version 0.3
Parts:
- removed B5, B6, B7, B8: (no value), PatternAgents-TouchWidgets:BUTTON_PASSIVE_12MM
- removed LED1, LED2, LED3, LED4: (no value), adafruit:CHIP-LED0805
- removed SJ1, SJ3, SJ5, SJ7: AHLB, SparkFun-Passives:PAD-JUMPER-2-NO_YES_SILK
- removed SJ2, SJ4, SJ6, SJ8: TOG, SparkFun-Passives:PAD-JUMPER-2-NO_YES_SILK
- added BTN1, BTN2, BTN3, BTN4: BUTTON_PASSIVE_LED, My Eagle Lib:BUTTON_PASSIVE_LED
- moved C4 26.7 mm to (38.1, 30.5), turned to 0 degrees
- moved U$2 19.9 mm to (35.6, 34.9)
- moved C1 19.6 mm to (38.2, 27.2)
- moved R2 18.8 mm to (34.9, 41.9), turned to 0 degrees
- moved C2 18.2 mm to (31.9, 27.2)
- moved C3 17.5 mm to (31.8, 30.5), turned to 180 degrees
- moved R1 17.3 mm to (34.9, 16.5), turned to 0 degrees
- moved U$1 16.0 mm to (35.6, 22.9)
- moved C7 13.1 mm to (50.2, 30.5)
- moved C8 12.8 mm to (43.8, 30.5)
- moved U$4 12.1 mm to (47.0, 34.9)
- moved R4 9.09 mm to (47.6, 41.9)
- moved C5 7.56 mm to (50.2, 27.2)
- moved C6 7.00 mm to (43.9, 27.2)
- moved R3 5.43 mm to (47.6, 16.5)
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Connections:
- removed net N$1: SJ1.1, U$1.4
- removed net N$11: SJ5.1, U$3.4
- removed net N$12: SJ6.1, U$3.6
- removed net N$15: SJ7.1, U$4.4
- removed net N$16: SJ8.1, U$4.6
- removed net N$3: LED1.A, R1.2
- removed net N$4: LED2.A, R2.2
- removed net N$5: SJ2.1, U$1.6
- removed net N$6: LED3.A, R3.2
- removed net N$7: SJ3.1, U$2.4
- removed net N$8: SJ4.1, U$2.6
- removed net N$9: LED4.A, R4.2
- new net N$10: BTN1.A, R1.2
- new net N$13: BTN2.A, R2.2
- new net N$14: BTN3.A, R3.2
- new net N$17: BTN4.A, R4.2
- net D1: now also BTN1.C; no longer LED1.C
- net D2: now also BTN2.C; no longer LED2.C
- net D3: now also BTN3.C; no longer LED3.C
- net D4: now also BTN4.C; no longer LED4.C
- net I1: now also BTN1.BUTTON; no longer B5.BUTTON
- net I2: now also BTN2.BUTTON; no longer B6.BUTTON
- net I3: now also BTN3.BUTTON; no longer B7.BUTTON
- net I4: now also BTN4.BUTTON; no longer B8.BUTTON
- net VDD: no longer SJ1.2, SJ2.2, SJ3.2, SJ4.2, SJ5.2, SJ6.2, SJ7.2, SJ8.2
Routing:
- net GND: track 125.5 -> 91.1 mm, vias 1 -> 2
- net VDD: track 142.5 -> 113.1 mm, vias 2 -> 3
- net D5: track 23.2 -> 39.4 mm, vias 1 -> 2
- net D7: track 61.4 -> 76.3 mm
- net D3: track 68.7 -> 81.5 mm, vias 0 -> 1
- net N$17: track 0.00 -> 11.1 mm
- net N$10: track 0.00 -> 10.4 mm
- net D0: track 25.1 -> 34.9 mm, vias 0 -> 1
- net N$13: track 0.00 -> 8.51 mm
- net N$14: track 0.00 -> 7.72 mm
- net N$4: track 5.68 -> 0.00 mm, vias 1 -> 0
- net N$9: track 5.33 -> 0.00 mm, vias 1 -> 0
- net D2: track 25.6 -> 30.8 mm, vias 1 -> 0
- net N$3: track 4.69 -> 0.00 mm, vias 1 -> 0
- net N$6: track 4.69 -> 0.00 mm, vias 1 -> 0
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Other:
- board text added: "Rocky Switch Shield v0.3"
- board text removed: "Rocky Switch Shield v0.2"

Commit message: Update to version 0.4
Parts:
- moved U$3 19.7 mm to (66.7, 21.6)
- moved U$4 19.7 mm to (66.7, 34.3)
- moved C8 18.0 mm to (61.8, 29.8)
- moved C6 17.9 mm to (61.8, 26.2)
- moved C5 17.2 mm to (67.3, 26.2)
- moved C7 17.2 mm to (67.3, 29.8)
- moved C3 14.9 mm to (46.4, 33.7), turned to 0 degrees
- moved U$2 13.9 mm to (48.3, 29.2)
- moved R1 7.24 mm to (40.6, 12.1)
- moved U$1 6.48 mm to (41.9, 21.6)
- moved C2 6.43 mm to (38.2, 26.2)
- moved R2 6.25 mm to (40.6, 44.5)
- moved BTN1 5.71 mm to (30.5, 17.1)
- moved BTN2 5.71 mm to (30.5, 39.4)
- moved C1 5.18 mm to (43.3, 26.2)
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Connections:
- net D0: now also U$4.1; no longer U$1.1
- net D5: now also U$3.1; no longer U$2.1
- net D6: now also U$2.1; no longer U$3.1
- net D7: now also U$1.1; no longer U$4.1
Routing:
- net VDD: track 113.1 -> 168.7 mm, vias 3 -> 4
- net D0: track 34.9 -> 72.6 mm
- net D7: track 76.3 -> 38.8 mm, vias 1 -> 2
- net GND: track 91.1 -> 118.6 mm, vias 2 -> 4
- net D5: track 39.4 -> 65.8 mm
- net I2: track 15.2 -> 22.7 mm
- net D3: track 81.5 -> 75.2 mm, vias 1 -> 0
- net I3: track 12.5 -> 18.7 mm
- net D1: track 26.2 -> 31.5 mm
- net N$14: track 7.72 -> 12.0 mm
- net I4: track 10.7 -> 14.1 mm
- net I1: track 16.2 -> 19.2 mm, vias 0 -> 2
- net D4: track 61.2 -> 64.0 mm, vias 1 -> 2
- net D2: track 30.8 -> 33.5 mm, vias 0 -> 1
- net N$17: track 11.1 -> 13.5 mm
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Other:
- board text added: "Rocky Switch Shield v0.4"
- board text removed: "Rocky Switch Shield v0.3"

Commit message: Update design to v0.5
Parts:
- C1, C3, C5, C7: value 30pF -> 10pF
Other:
- board text added: "Rocky Switch Shield v0.5"
- board text removed: "Rocky Switch Shield v0.4"
Changed lines of the file:
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@@
 <text x="4.699" y="32.258" size="1.016" layer="25" font="vector" ratio="15" rot="SR90">D1</text>
 <text x="4.699" y="34.798" size="1.016" layer="25" font="vector" ratio="15" rot="SR90">D2</text>
-<text x="22.225" y="5.588" size="1.524" layer="25" font="vector" ratio="20" rot="SR0">Rocky Switch Shield v0.4</text>
+<text x="22.225" y="5.588" size="1.524" layer="25" font="vector" ratio="20" rot="SR0">Rocky Switch Shield v0.5</text>
 <text x="4.699" y="37.338" size="1.016" layer="25" font="vector" ratio="15" rot="SR90">D3</text>
 <text x="4.699" y="39.878" size="1.016" layer="25" font="vector" ratio="15" rot="SR90">D4</text>
@@
 <attribute name="VALUE" x="12.065" y="31.75" size="1.27" layer="27" rot="R90"/>
 </element>
-<element name="C1" library="rcl" package="C0805K" value="30pF" x="43.307" y="26.162" smashed="yes" rot="MR0">
+<element name="C1" library="rcl" package="C0805K" value="10pF" x="43.307" y="26.162" smashed="yes" rot="MR0">
 <attribute name="NAME" x="41.289" y="26.908" size="0.762" layer="26" font="vector" ratio="15" rot="MR270"/>
 <attribute name="VALUE" x="44.434" y="27.31" size="0.762" layer="28" font="vector" ratio="15" rot="MR0"/>
@@
 <attribute name="VALUE" x="39.608" y="27.31" size="0.762" layer="28" font="vector" ratio="15" rot="MR0"/>
 </element>
-<element name="C3" library="rcl" package="C0805K" value="30pF" x="46.355" y="33.655" smashed="yes" rot="MR0">
+<element name="C3" library="rcl" package="C0805K" value="10pF" x="46.355" y="33.655" smashed="yes" rot="MR0">
 <attribute name="NAME" x="49.036" y="34.401" size="0.762" layer="26" font="vector" ratio="15" rot="MR270"/>
 <attribute name="VALUE" x="47.609" y="34.93" size="0.762" layer="28" font="vector" ratio="15" rot="MR0"/>
@@
 <attribute name="VALUE" x="39.386" y="35.682" size="0.762" layer="28" font="vector" ratio="15" rot="MR180"/>
 </element>
-<element name="C5" library="rcl" package="C0805K" value="30pF" x="67.31" y="26.162" smashed="yes" rot="MR0">
+<element name="C5" library="rcl" package="C0805K" value="10pF" x="67.31" y="26.162" smashed="yes" rot="MR0">
 <attribute name="NAME" x="65.292" y="26.781" size="0.762" layer="26" font="vector" ratio="15" rot="MR270"/>
 <attribute name="VALUE" x="68.31" y="27.437" size="0.762" layer="28" font="vector" ratio="15" rot="MR0"/>
@@
 <attribute name="VALUE" x="63.103" y="27.437" size="0.762" layer="28" font="vector" ratio="15" rot="MR0"/>
 </element>
-<element name="C7" library="rcl" package="C0805K" value="30pF" x="67.31" y="29.845" smashed="yes" rot="MR0">
+<element name="C7" library="rcl" package="C0805K" value="10pF" x="67.31" y="29.845" smashed="yes" rot="MR0">
 <attribute name="NAME" x="65.292" y="30.591" size="0.762" layer="26" font="vector" ratio="15" rot="MR270"/>
 <attribute name="VALUE" x="68.437" y="31.247" size="0.762" layer="28" font="vector" ratio="15" rot="MR0"/>

Commit message: Update design to version 1.0
Other:
- board text added: "Rocky Switch Shield v1.0"
- board text removed: "Rocky Switch Shield v0.5"
Changed lines of the file:
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@@
 <text x="4.699" y="32.258" size="1.016" layer="25" font="vector" ratio="15" rot="SR90">D1</text>
 <text x="4.699" y="34.798" size="1.016" layer="25" font="vector" ratio="15" rot="SR90">D2</text>
-<text x="22.225" y="5.588" size="1.524" layer="25" font="vector" ratio="20" rot="SR0">Rocky Switch Shield v0.5</text>
+<text x="22.225" y="5.588" size="1.524" layer="25" font="vector" ratio="20" rot="SR0">Rocky Switch Shield v1.0</text>
 <text x="4.699" y="37.338" size="1.016" layer="25" font="vector" ratio="15" rot="SR90">D3</text>
 <text x="4.699" y="39.878" size="1.016" layer="25" font="vector" ratio="15" rot="SR90">D4</text>
