File: Rocky Switch Shield.sch (EAGLE design)
At the start: 10 parts

Commit message: Update new shield for rocky switch
Parts:
- removed CAP_BTN1, CAP_BTN2, CAP_BTN3: (no value), adafruit:PINHD-1X3
- removed JP2: (no value), adafruit:PINHD-2X4
- added B5, B6, B7, B8: (no value), PatternAgents-TouchWidgets:BUTTON_PASSIVE12MM
- added C1, C3, C5, C7: 30pF, rcl:C-EUC0805K
- added C2, C4, C6, C8: 0.1uF, rcl:C-EUC0805K
- added JP1: (no value), pinhead:PINHD-2X5
- added LED4: (no value), adafruit:LED3MM
- added R4: 1K, rcl:R-EU_R0805
- added SJ1, SJ2, SJ3, SJ4, SJ5, SJ6, SJ7, SJ8: JUMPER-PAD-2-NOYES_SILK, SparkFun-Passives:JUMPER-PAD-2-NOYES_SILK
- added U$1, U$2, U$3, U$4: TTP223B, My Eagle Lib:TTP223B
Connections:
- removed net 3V3: CAP_BTN1.3, CAP_BTN2.3, CAP_BTN3.3, JP2.1
- new net D3: JP1.6, LED3.C
- new net D4: JP1.8, LED4.C
- new net I1: B5.BUTTON, C1.1, U$1.I
- new net I2: B6.BUTTON, C3.1, U$2.I
- new net I3: B7.BUTTON, C5.1, U$3.I
- new net I4: B8.BUTTON, C7.1, U$4.I
- new net N$1: SJ1.1, U$1.TOG
- new net N$11: SJ5.1, U$3.TOG
- new net N$12: SJ6.1, U$3.AHLB
- new net N$15: SJ7.1, U$4.TOG
- new net N$16: SJ8.1, U$4.AHLB
- new net N$5: SJ2.1, U$1.AHLB
- new net N$7: SJ3.1, U$2.TOG
- new net N$8: SJ4.1, U$2.AHLB
- new net N$9: LED4.A, R4.2
- new net VDD: C2.1, C4.1, C6.1, C8.1, JP1.10, R1.1, R2.1, R3.1, R4.1, SJ1.2, SJ2.2, SJ3.2, SJ4.2, SJ5.2, SJ6.2, SJ7.2, SJ8.2, U$1.VDD, U$2.VDD, U$3.VDD, U$4.VDD
- net D0: now also JP1.7, U$1.Q; no longer CAP_BTN1.2, JP2.4
- net D1: now also JP1.2, LED1.C; no longer CAP_BTN2.2, JP2.6
- net D2: now also JP1.4, LED2.C; no longer CAP_BTN3.2, JP2.8
- net D5: now also JP1.5, U$2.Q; no longer JP2.7, R3.1
- net D6: now also JP1.3, U$3.Q; no longer JP2.5, R2.1
- net D7: now also JP1.1, U$4.Q; no longer JP2.3, R1.1
- net GND: now also C1.2, C2.2, C3.2, C4.2, C5.2, C6.2, C7.2, C8.2, JP1.9, U$1.VSS, U$2.VSS, U$3.VSS, U$4.VSS; no longer CAP_BTN1.1, CAP_BTN2.1, CAP_BTN3.1, JP2.2, LED1.C, LED2.C, LED3.C
Other:
- moved on the sheet: LED1, LED2, LED3, R1, R2, R3

Commit message: Update board design to version 0.2
Parts:
- LED1, LED2, LED3, LED4: device adafruit:LED3MM -> adafruit:LEDCHIP-LED0805
- SJ1, SJ3, SJ5, SJ7: value JUMPER-PAD-2-NOYES_SILK -> AHLB
- SJ2, SJ4, SJ6, SJ8: value JUMPER-PAD-2-NOYES_SILK -> TOG
Other:
- note added: "2016-10-09 http://easytech.vn"
- note added: "AHLB=Output active high or low selection High=Active low output Low=Active high output"
- note added: "Capacitive Buttons"
- note added: "Rocky Switch Shield v0.2"
- note added: "TOG=Output type option pin High=Toggle mode (On/Off) Low=Momentary mode (ON pulse when touch)"
- moved on the sheet: B5, B6, B7, B8, C1, C2, C3, C4, C5, C6, C7, C8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

Commit message: Update design to version 0.3
Parts:
- removed B5, B6, B7, B8: (no value), PatternAgents-TouchWidgets:BUTTON_PASSIVE12MM
- removed LED1, LED2, LED3, LED4: (no value), adafruit:LEDCHIP-LED0805
- removed SJ1, SJ3, SJ5, SJ7: AHLB, SparkFun-Passives:JUMPER-PAD-2-NOYES_SILK
- removed SJ2, SJ4, SJ6, SJ8: TOG, SparkFun-Passives:JUMPER-PAD-2-NOYES_SILK
- added BTN1, BTN2, BTN3, BTN4: BUTTON_PASSIVE_LED, My Eagle Lib:BUTTON_PASSIVE_LED
Connections:
- removed net N$1: SJ1.1, U$1.TOG
- removed net N$11: SJ5.1, U$3.TOG
- removed net N$12: SJ6.1, U$3.AHLB
- removed net N$15: SJ7.1, U$4.TOG
- removed net N$16: SJ8.1, U$4.AHLB
- removed net N$3: LED1.A, R1.2
- removed net N$4: LED2.A, R2.2
- removed net N$5: SJ2.1, U$1.AHLB
- removed net N$6: LED3.A, R3.2
- removed net N$7: SJ3.1, U$2.TOG
- removed net N$8: SJ4.1, U$2.AHLB
- removed net N$9: LED4.A, R4.2
- new net N$10: BTN1.A, R1.2
- new net N$13: BTN2.A, R2.2
- new net N$14: BTN3.A, R3.2
- new net N$17: BTN4.A, R4.2
- net D1: now also BTN1.C; no longer LED1.C
- net D2: now also BTN2.C; no longer LED2.C
- net D3: now also BTN3.C; no longer LED3.C
- net D4: now also BTN4.C; no longer LED4.C
- net I1: now also BTN1.BUTTON; no longer B5.BUTTON
- net I2: now also BTN2.BUTTON; no longer B6.BUTTON
- net I3: now also BTN3.BUTTON; no longer B7.BUTTON
- net I4: now also BTN4.BUTTON; no longer B8.BUTTON
- net VDD: no longer SJ1.2, SJ2.2, SJ3.2, SJ4.2, SJ5.2, SJ6.2, SJ7.2, SJ8.2
Other:
- note added: "2016-10-17 http://easytech.vn"
- note added: "Rocky Switch Shield v0.3"
- note removed: "2016-10-09 http://easytech.vn"
- note removed: "Rocky Switch Shield v0.2"
- moved on the sheet: C1, C3, C4, C5, C6, C7, C8, JP1, R1, R2, R3, R4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

Commit message: Update to version 0.4
Connections:
- net D0: now also U$4.Q; no longer U$1.Q
- net D5: now also U$3.Q; no longer U$2.Q
- net D6: now also U$2.Q; no longer U$3.Q
- net D7: now also U$1.Q; no longer U$4.Q
Other:
- note added: "Rocky Switch Shield v0.4"
- note removed: "Rocky Switch Shield v0.3"
- moved on the sheet: C2, C4, C6, C8, JP1

Commit message: Update design to v0.5
Parts:
- C1, C3, C5, C7: value 30pF -> 10pF
Other:
- note added: "2016-10-24 http://easytech.vn"
- note added: "Rocky Switch Shield v0.5"
- note removed: "2016-10-17 http://easytech.vn"
- note removed: "Rocky Switch Shield v0.4"
- moved on the sheet: C2, C4, C6, C8, JP1

Commit message: Update design to version 1.0
Other:
- note added: "Rocky Switch Shield v1.0"
- note removed: "Rocky Switch Shield v0.5"
Changed lines of the file:
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@@
 <wire x1="203.2" y1="-38.1" x2="-25.4" y2="-38.1" width="0.1524" layer="97"/>
 <wire x1="-25.4" y1="-38.1" x2="-25.4" y2="144.78" width="0.1524" layer="97"/>
-<text x="99.06" y="134.62" size="5.08" layer="97" font="vector" ratio="15">Rocky Switch Shield v0.5</text>
+<text x="99.06" y="134.62" size="5.08" layer="97" font="vector" ratio="15">Rocky Switch Shield v1.0</text>
 <text x="99.06" y="124.46" size="2.54" layer="97" font="vector" ratio="15">2016-10-24
 http://easytech.vn</text>
