File: Rocky Switch Relay Shield.sch (EAGLE design)
At the start: 21 parts

Commit message: Add shield for rocky relay
Parts:
- removed BTN1, BTN2, BTN3, BTN4: BUTTON_PASSIVE_LED, My Eagle Lib:BUTTON_PASSIVE_LED
- removed C7: 10pF, rcl:C-EUC0805K
- removed C8: 0.1uF, rcl:C-EUC0805K
- removed JP1: (no value), pinhead:PINHD-2X5
- removed R4: 1K, rcl:R-EU_R0805
- removed U$1, U$2, U$3, U$4: TTP223B, My Eagle Lib:TTP223B
- added BUTTON1, BUTTON2, BUTTON3: BUTTON_PASSIVE_LED, My Eagle Lib:BUTTON_PASSIVE_LED
- added JP2: (no value), pinhead:PINHD-2X4
- added U$16, U$18, U$19: TTP223B, My Eagle Lib:TTP223B
Connections:
- removed net D0: JP1.7, U$4.Q
- removed net D4: BTN4.C, JP1.8
- removed net I4: BTN4.BUTTON, C7.1, U$4.I
- removed net N$13: BTN2.A, R2.2
- removed net N$14: BTN3.A, R3.2
- removed net N$17: BTN4.A, R4.2
- removed net VDD: C2.1, C4.1, C6.1, C8.1, JP1.10, R1.1, R2.1, R3.1, R4.1, U$1.VDD, U$2.VDD, U$3.VDD, U$4.VDD
- new net 5V: C2.1, C4.1, C6.1, JP2.1, R1.1, R2.1, R3.1, U$16.VDD, U$18.VDD, U$19.VDD
- new net N$15: BUTTON2.A, R2.2
- new net N$16: BUTTON3.A, R3.2
- net D1: now also BUTTON1.C, JP2.7; no longer BTN1.C, JP1.2
- net D2: now also BUTTON2.C, JP2.5; no longer BTN2.C, JP1.4
- net D3: now also BUTTON3.C, JP2.3; no longer BTN3.C, JP1.6
- net D5: now also JP2.8, U$19.Q; no longer JP1.5, U$3.Q
- net D6: now also JP2.6, U$18.Q; no longer JP1.3, U$2.Q
- net D7: now also JP2.4, U$16.Q; no longer JP1.1, U$1.Q
- net GND: now also JP2.2, U$16.VSS, U$18.VSS, U$19.VSS; no longer C7.2, C8.2, JP1.9, U$1.VSS, U$2.VSS, U$3.VSS, U$4.VSS
- net I1: now also BUTTON1.BUTTON, U$16.I; no longer BTN1.BUTTON, U$1.I
- net I2: now also BUTTON2.BUTTON, U$18.I; no longer BTN2.BUTTON, U$2.I
- net I3: now also BUTTON3.BUTTON, U$19.I; no longer BTN3.BUTTON, U$3.I
- net N$10: now also BUTTON1.A; no longer BTN1.A
Other:
- note added: "2017-06-09 http://easytech.vn"
- note added: "Rocky Switch Shield v2.0"
- note removed: "2016-10-24 http://easytech.vn"
- note removed: "Rocky Switch Shield v1.0"
- moved on the sheet: C1, C2, C3, C4, C5, C6, R1, R2, R3
